File: cw key.kicad_sch (KiCad schematic)
At the start: 32 parts, among them J1 AudioPlug3, J2 Conn_01x01_Pin, J3 Conn_01x01_Pin, J4 Conn_ARM_SWD_TagConnect_TC203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, J5 AudioPlug3, SW3 SW_SPST, U1 MSPM0C1103SDSGR, U2 MTCH1030

Commit message: melted
Parts:
- added J6, J7: Conn_01x01_Pin, footprints:Header_spacer, symbol Connector:Conn_01x01_Pin
- J1, J5: footprint footprints:3.5 mm plug -> footprints:3.5 mm plug 4 pin
Connections:
- net GND_shield: now also J7.1 (Pin_1)
- net pad_0: now also J6.1 (Pin_1)
Other:
- removed sheet touch pad
Changed lines of the file:
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@@
 	(wire
 		(pts
-			(xy 59.69 85.09) (xy 59.69 102.87)
+			(xy 59.69 85.09) (xy 59.69 87.63)
 		)
 		(stroke
@@
 	(wire
 		(pts
-			(xy 43.18 95.25) (xy 43.18 74.93)
+			(xy 43.18 77.47) (xy 43.18 74.93)
 		)
 		(stroke
@@
 	(wire
 		(pts
-			(xy 38.1 95.25) (xy 43.18 95.25)
-		)
-		(stroke
-			(width 0)
-			(type default)
-		)
-	)
-	(wire
-		(pts
 			(xy 237.49 129.54) (xy 237.49 114.3)
 		)
@@
 	(wire
 		(pts
-			(xy 38.1 102.87) (xy 59.69 102.87)
-		)
-		(stroke
-			(width 0)
-			(type default)
-		)
-	)
-	(wire
-		(pts
 			(xy 231.14 44.45) (xy 233.68 44.45)
 		)
@@
 			)
 		)
-		(property "Footprint" "footprints:3.5 mm plug"
+		(property "Footprint" "footprints:3.5 mm plug 4 pin"
 			(at 255.27 128.27 0)
 			(effects
@@
 			)
 		)
-		(property "Footprint" "footprints:3.5 mm plug"
+		(property "Footprint" "footprints:3.5 mm plug 4 pin"
 			(at 255.27 113.03 0)
 			(effects
@@
 	)
 	(symbol
+		(lib_id "Connector:Conn_01x01_Pin")
+		(at 38.1 77.47 0)
+		(unit 1)
+		(exclude_from_sim no)
+		(in_bom yes)
+		(on_board yes)
+		(dnp no)
+		(property "Reference" "J6"
+			(at 36.068 77.47 0)
+			(effects
+				(font
+					(size 1.27 1.27)
+				)
+			)
+		)
+		(property "Value" "Conn_01x01_Pin"
+			(at 38.735 74.93 0)
+			(effects
+				(font
+					(size 1.27 1.27)
+				)
+				(hide yes)
+			)
+		)
+		(property "Footprint" "footprints:Header_spacer"
+			(at 38.1 77.47 0)
+			(effects
+				(font
+					(size 1.27 1.27)
+				)
+				(hide yes)
+			)
+		)
+		(property "Datasheet" "~"
+			(at 38.1 77.47 0)
+			(effects
+				(font
+					(size 1.27 1.27)
+				)
+				(hide yes)
+			)
+		)
+		(property "Description" "Generic connector, single row, 01x01, script generated"
+			(at 38.1 77.47 0)
+			(effects
+				(font
+					(size 1.27 1.27)
+				)
+				(hide yes)
+			)
+		)
+		(pin "1"
+		)
+		(instances
+			(project "cw key"
+				(path "/a794b037-5597-4c1c-8f69-6ec2c837a701"
+					(reference "J6")
+					(unit 1)
+				)
+			)
+		)
+	)
+	(symbol
 		(lib_id "power:GND")
 		(at 193.04 158.75 0)
@@
 	)
 	(symbol
+		(lib_id "Connector:Conn_01x01_Pin")
+		(at 54.61 87.63 0)
+		(unit 1)
+		(exclude_from_sim no)
+		(in_bom yes)
+		(on_board yes)
+		(dnp no)
+		(property "Reference" "J7"
+			(at 52.578 87.63 0)
+			(effects
+				(font
+					(size 1.27 1.27)
+				)
+			)
+		)
+		(property "Value" "Conn_01x01_Pin"
+			(at 55.245 85.09 0)
+			(effects
+				(font
+					(size 1.27 1.27)
+				)
+				(hide yes)
+			)
+		)
+		(property "Footprint" "footprints:Header_spacer"
+			(at 54.61 87.63 0)
+			(effects
+				(font
+					(size 1.27 1.27)
+				)
+				(hide yes)
+			)
+		)
+		(property "Datasheet" "~"
+			(at 54.61 87.63 0)
+			(effects
+				(font
+					(size 1.27 1.27)
+				)
+				(hide yes)
+			)
+		)
+		(property "Description" "Generic connector, single row, 01x01, script generated"
+			(at 54.61 87.63 0)
+			(effects
+				(font
+					(size 1.27 1.27)
+				)
+				(hide yes)
+			)
+		)
+		(pin "1"
+		)
+		(instances
+			(project "cw key"
+				(path "/a794b037-5597-4c1c-8f69-6ec2c837a701"
+					(reference "J7")
+					(unit 1)
+				)
+			)
+		)
+	)
+	(symbol
 		(lib_id "power:GND")
 		(at 77.47 154.94 0)
@@
 				)
 			)
-		)
-	)
-	(sheet
-		(at 16.51 90.17)
-		(size 21.59 19.05)
-		(exclude_from_sim no)
-		(in_bom yes)
-		(on_board yes)
-		(dnp no)
-		(fields_autoplaced yes)
-		(stroke
-			(width 0.1524)
-			(type solid)
-		)
-		(fill
-			(color 0 0 0 0.0000)
-		)
-		(property "Sheetname" "touch pad"
-			(at 16.51 89.4584 0)
-			(effects
-				(font
-					(size 1.27 1.27)
-				)
-				(justify left bottom)
-			)
-		)
-		(property "Sheetfile" "touch pad.kicad_sch"
-			(at 16.51 109.8046 0)
-			(effects
-				(font
-					(size 1.27 1.27)
-				)
-				(justify left top)
-			)
-		)
-		(pin "GND_shield" input
-			(at 38.1 102.87 0)
-			(effects
-				(font
-					(size 1.27 1.27)
-				)
-				(justify right)
-			)
-		)
-		(pin "pad 0" input
-			(at 38.1 95.25 0)
-			(effects
-				(font
-					(size 1.27 1.27)
-				)
-				(justify right)
-			)
-		)
-		(instances
-			(project "cw key"
-				(path "/a794b037-5597-4c1c-8f69-6ec2c837a701"
-					(page "2")
-				)
-			)
